Commit message: moved components into main xacro

File: bounce/xacro/bounce.xacro (robot description, xacro)
@@ -2,4 +2,58 @@
 <sdf version="1.7"
     xmlns:xacro="http://www.ros.org/wiki/xacro">
+    <!-- balls are modeled as spherical shells with bounce -->
+    <xacro:macro name="ball" params="name bounce color mass:=1 radius:=0.25 *pose">
+        <model name="${name}">
+            <xacro:insert_block name="pose" />
+            <link name="${name}_link">
+                <pose>0 0 ${radius} 0 0 0</pose>
+                <inertial>
+                    <pose>0 0 0 0 0 0</pose>
+                    <mass>${mass}</mass>
+                    <inertia>
+                        <ixx>${2/3 * mass * radius * radius}</ixx>
+                        <ixy>0</ixy>
+                        <ixz>0</ixz>
+                        <iyy>${2/3 * mass * radius * radius}</iyy>
+                        <iyz>0</iyz>
+                        <izz>${2/3 * mass * radius * radius}</izz>
+                    </inertia>
+                </inertial>
+                <collision name="${name}_collision">
+                    <pose relative_to="${name}_link">0 0 0 0 0 0</pose>
+                    <geometry>
+                        <sphere>
+                            <radius>${radius}</radius>
+                        </sphere>
+                    </geometry>
+                    <surface>
+                        <bounce>
+                            <restitution_coefficient>${bounce}</restitution_coefficient>
+                            <threshold>0</threshold>
+                        </bounce>
+                        <contact>
+                            <ode>
+                                <max_vel>1000</max_vel>
+                            </ode>
+                        </contact>
+                    </surface>
+                </collision>
+                <visual name="${name}_visual">
+                    <pose>0 0 0 0 0 0</pose>
+                    <geometry>
+                        <sphere>
+                            <radius>${radius}</radius>
+                        </sphere>
+                    </geometry>
+                    <material>
+                        <ambient>${color}</ambient>
+                        <diffuse>${color}</diffuse>
+                        <specular>0.1 0.1 0.1 1</specular>
+                    </material>
+                </visual>
+                <gravity>1</gravity>
+            </link>
+        </model>
+    </xacro:macro>
     <!-- A ground plane -->
     <xacro:macro name="ground_plane">

File: bounce/xacro/bounce_test.xacro (robot description, xacro)
@@ -6,6 +6,5 @@
     <plugin filename="gz-sim-user-commands-system" name="gz::sim::systems::UserCommands" />
     <plugin filename="gz-sim-scene-broadcaster-system" name="gz::sim::systems::SceneBroadcaster" />
-    <xacro:include filename="balls.xacro" />
-    <xacro:include filename="world_components.xacro" />
+    <xacro:include filename="bounce.xacro" />
     <xacro:ground_plane/>
     <xacro:sun/>
